File: discipline_iso/discipline-pcb.sch (KiCad schematic (older format))
At the start: 165 parts, among them J1 AVR-ISP-6, SW1 KEYSW, SW10 KEYSW, SW11 KEYSW, SW12 KEYSW, SW13 KEYSW, SW14 KEYSW, SW15 KEYSW, SW16 KEYSW, SW17 KEYSW, SW18 KEYSW, SW19 KEYSW, SW2 KEYSW, SW20 KEYSW, SW21 KEYSW, SW22 KEYSW, SW23 KEYSW, SW24 KEYSW, SW25 KEYSW, SW26 KEYSW, SW27 KEYSW, SW28 KEYSW, SW29 KEYSW, SW3 KEYSW, SW30 KEYSW, SW31 KEYSW, SW310 KEYSW, SW32 KEYSW, SW33 KEYSW, SW34 KEYSW, SW35 KEYSW, SW36 KEYSW, SW37 KEYSW, SW38 KEYSW, SW39 KEYSW, SW4 KEYSW, SW40 KEYSW, SW41 KEYSW, SW42 KEYSW, SW43 KEYSW, SW44 KEYSW, SW45 KEYSW, SW46 KEYSW, SW47 KEYSW, SW48 KEYSW, SW49 KEYSW, SW5 KEYSW, SW50 KEYSW, SW51 KEYSW, SW52 KEYSW, SW53 KEYSW, SW54 KEYSW, SW55 KEYSW, SW56 KEYSW, SW57 KEYSW, SW58 KEYSW, SW59 KEYSW, SW590 KEYSW, SW6 KEYSW, SW60 KEYSW, SW61 KEYSW, SW610 KEYSW, SW62 KEYSW, SW620 KEYSW, SW63 KEYSW, SW630 KEYSW, SW64 KEYSW, SW640 KEYSW, SW65 KEYSW, SW66 KEYSW, SW67 KEYSW, SW68 KEYSW, SW69 KEYSW, SW7 KEYSW, SW8 KEYSW, SW9 KEYSW, U1 ATmega32A-PU, Y1 Crystal

Commit message: Add files via upload
Parts:
- added D690: (no value), Diode_THT:D_T-1_P5.08mm_Horizontal, symbol Device:D
Connections:
- net row3: now also D690.1 (K); no longer SW69.2
- new net: D690.2 (A), SW69.2
Changed lines of the file:
@@
 	2850 5050 2900 5050
 Connection ~ 2900 5050
-Wire Wire Line
-	2900 5050 3650 5050
 Text Label 2850 5050 0    50   ~ 0
 row3
@@
 Wire Wire Line
 	4250 4700 4250 5250
-Wire Wire Line
-	3650 4700 3650 5050
-Connection ~ 3650 5050
-Wire Wire Line
-	3650 5050 4300 5050
 $Comp
 L discipline-pcb-rescue:KEYSW-keyboard_parts SW310
@@
 	1    0    0    -1
 $EndComp
+Wire Wire Line
+	2900 5050 3634 5050
+Wire Wire Line
+	3610 4700 3650 4700
+$Comp
+L Device:D D690
+U 1 1 5D9538D9
+P 3585 4867
+F 0 "D690" V 3631 4788 50  0000 R CNN
+F 1 " " V 3540 4788 50  0000 R CNN
+F 2 "Diode_THT:D_T-1_P5.08mm_Horizontal" H 3585 4867 50  0001 C CNN
+F 3 "~" H 3585 4867 50  0001 C CNN
+	1    3585 4867
+	0    -1   -1   0
+$EndComp
+Wire Wire Line
+	3585 5017 3634 5017
+Wire Wire Line
+	3634 5017 3634 5050
+Connection ~ 3634 5050
+Wire Wire Line
+	3634 5050 4300 5050
+Wire Wire Line
+	3585 4718 3585 4717
+Wire Wire Line
+	3585 4667 3610 4667
+Wire Wire Line
+	3610 4667 3610 4700
+Connection ~ 3585 4717
+Wire Wire Line
+	3585 4717 3585 4667
 $EndSCHEMATC
